Commit message: [fix] Need inertia in base_link to generate joint

File: colcon_ws/src/diffbot_description/robots/diffbot_description.urdf.xacro (robot description, xacro)
@@ -13,8 +13,8 @@
   <xacro:macro name="wheel_macro" params="parent prefix xyz">
     <joint name="${prefix}_joint" type="continuous">
-      <origin xyz="${xyz}" rpy="${radians(-90)} 0 0"/>
+      <axis xyz="0 0 1" />
       <parent link="${parent}"/>
       <child  link="${prefix}_link"/>
-      <axis xyz="0 0 1" />
+      <origin xyz="${xyz}" rpy="${radians(-90)} 0 0"/>
     </joint>
     <link name="${prefix}_link">
@@ -37,5 +37,11 @@
     </link>
   </xacro:macro>
-  <link name="base_link"/>
+  <link name="base_link">
+    <inertial>
+      <origin xyz="0 0 0" rpy="0 0 0"/>
+      <mass value="0.01"/>
+      <inertia ixx="0.0001" ixy="0.0" ixz="0.0" iyy="0.0001" iyz="0.0" izz="0.0001"/>
+    </inertial>
+  </link>
   <joint name="body_joint" type="fixed">
     <parent link="base_link"/>
@@ -63,10 +69,10 @@
     </collision>
   </link>
-  <xacro:wheel_macro prefix="left_wheel"  parent="base_link" xyz="0 0.1 0.05"/>
-  <xacro:wheel_macro prefix="right_wheel" parent="base_link" xyz="0 -0.1 0.05"/>
+  <xacro:wheel_macro prefix="left_wheel"  parent="body_link" xyz="0.07 0.1 -0.02"/>
+  <xacro:wheel_macro prefix="right_wheel" parent="body_link" xyz="0.07 -0.1 -0.02"/>
   <joint name="ball_joint" type="fixed">
-    <parent link="base_link"/>
+    <parent link="body_link"/>
     <child  link="ball_link"/>
-    <origin xyz="-0.14 0 0.04" rpy="0 0 0"/>
+    <origin xyz="-0.07 0 -0.05" rpy="0 0 0"/>
   </joint>
   <link name="ball_link">
@@ -74,5 +80,5 @@
       <origin xyz="0 0 0" rpy="0 0 0" />
       <geometry>
-        <sphere radius="0.04" />
+        <sphere radius="0.02" />
       </geometry>
       <material name="ball" />
@@ -81,14 +87,24 @@
       <origin xyz="0 0 0" rpy="0 0 0" />
       <geometry>
-        <sphere radius="0.04" />
+        <sphere radius="0.02" />
       </geometry>
     </collision>
+    <inertial>
+      <origin xyz="0 0 0" rpy="0 0 0"/>
+      <mass value="0.1"/>
+      <inertia ixx="0.0001" ixy="0.0" ixz="0.0" iyy="0.0001" iyz="0.0" izz="0.0001"/>
+    </inertial>
   </link>
   <joint name="lidar_joint" type="fixed">
-    <parent link="base_link"/>
+    <parent link="body_link"/>
     <child  link="lidar_link"/>
     <origin xyz="0 0 0.2" rpy="0 0 0"/>
   </joint>
   <link name="lidar_link">
+    <inertial>
+      <origin xyz="0 0 0" rpy="0 0 0"/>
+      <mass value="0.1"/>
+      <inertia ixx="0.0001" ixy="0.0" ixz="0.0" iyy="0.0001" iyz="0.0" izz="0.0001"/>
+    </inertial>
     <!-- If visual tag is enable, lidar's ray is blocked. -->
     <!--
@@ -103,9 +119,14 @@
   </link>
   <joint name="camera_joint" type="fixed">
-    <parent link="base_link"/>
+    <parent link="body_link"/>
     <child  link="camera_link"/>
     <origin xyz="0.05 -0.1 0.1" rpy="0 0 0"/>
   </joint>
   <link name="camera_link">
+    <inertial>
+      <origin xyz="0 0 0" rpy="0 0 0"/>
+      <mass value="0.1"/>
+      <inertia ixx="0.0001" ixy="0.0" ixz="0.0" iyy="0.0001" iyz="0.0" izz="0.0001"/>
+    </inertial>
     <!-- If visual tag is enable, camera's view is blocked. -->
     <!--
@@ -120,9 +141,14 @@
   </link>
   <joint name="depth_camera_joint" type="fixed">
-    <parent link="base_link"/>
+    <parent link="body_link"/>
     <child  link="depth_camera_link"/>
     <origin xyz="0.05 0.1 0.1" rpy="0 0 0"/>
   </joint>
   <link name="depth_camera_link">
+    <inertial>
+      <origin xyz="0 0 0" rpy="0 0 0"/>
+      <mass value="0.1"/>
+      <inertia ixx="0.0001" ixy="0.0" ixz="0.0" iyy="0.0001" iyz="0.0" izz="0.0001"/>
+    </inertial>
     <!-- If visual tag is enable, camera's view is blocked. -->
     <!--
