Commit message: [add] add CameraMover.cs

File: colcon_ws/src/diffbot_description/robots/diffbot.urdf.xacro (robot description, xacro)
@@ -12,4 +12,6 @@
   <xacro:diffbot_ros2_control
     name="diffbot" prefix="$(arg prefix)" use_sim="$(arg use_sim)" />
+<!--
   <xacro:diffbot_isaac prefix="$(arg prefix)"/>
+-->
 </robot>

File: colcon_ws/src/diffbot_description/robots/diffbot_description.urdf.xacro (robot description, xacro)
@@ -4,13 +4,10 @@
   <material name="gray">
     <color rgba="0.5 0.5 0.5 0.2"/>
-    <isaac_rigid_body static_friction="0.8" dynamic_friction="0.5"/>
   </material>
   <material name="ball">
     <color rgba="0.5 0.5 0.5 0.2"/>
-    <isaac_rigid_body static_friction="0.0" dynamic_friction="0.0"/>
   </material>
   <material name="white">
     <color rgba="1.0 1.0 1.0 1.0"/>
-    <isaac_rigid_body static_friction="1.0" dynamic_friction="1.0"/>
   </material>
   <xacro:macro name="wheel_macro" params="parent prefix xyz">
@@ -20,15 +17,5 @@
       <child  link="${prefix}_link"/>
       <axis xyz="0 0 1" />
-      <isaac_drive_api stiffness="0" damping="30000" joint_friction="10000"/>
     </joint>
-    <transmission name="${prefix}_trans" type="SimpleTransmission">
-      <type>transmission_interface/SimpleTransmission</type>
-        <actuator name="${prefix}_motor">
-          <mechanicalReduction>50</mechanicalReduction>
-        </actuator>
-      <joint name="${prefix}_joint">
-        <hardwareInterface>hardware_interface/VelocityJointInterface</hardwareInterface>
-      </joint>
-    </transmission>
     <link name="${prefix}_link">
       <inertial>

Commit message: [change] change URDF to add sensor [remove] remove script for isaac sim

File: colcon_ws/src/diffbot_description/robots/diffbot.urdf.xacro (robot description, xacro)
@@ -8,10 +8,8 @@
   <xacro:include filename="$(find diffbot_description)/ros2_control/diffbot.ros2_control.xacro" />
   <!-- Import diffbot isaac description -->
-  <xacro:include filename="$(find diffbot_description)/isaac/diffbot.isaac.xacro" />
+  <xacro:include filename="$(find diffbot_description)/unity/diffbot.unity.xacro" />
   <xacro:diffbot prefix="$(arg prefix)" use_sim="$(arg use_sim)"/>
   <xacro:diffbot_ros2_control
     name="diffbot" prefix="$(arg prefix)" use_sim="$(arg use_sim)" />
-<!--
-  <xacro:diffbot_isaac prefix="$(arg prefix)"/>
--->
+  <xacro:diffbot_unity prefix="$(arg prefix)"/>
 </robot>

File: colcon_ws/src/diffbot_description/unity/diffbot.unity.xacro (robot description, xacro)
@@ -1,7 +1,7 @@
 <?xml version="1.0"?>
 <robot xmlns:xacro="http://ros.org/wiki/xacro">
-  <xacro:macro name="diffbot_isaac" params="prefix">
+  <xacro:macro name="diffbot_unity" params="prefix">
     <!-- =============== Isaac Sim =============== -->
-    <isaac>
+    <unity>
       <sensor name="lidar_link" type="lidar">
         <topic>scan</topic>
@@ -48,19 +48,5 @@
         <update_rate>10</update_rate>
       </sensor>
-      <surface_gripper name="body_link">
-        <topic>gripper_enable</topic>
-        <offset_x>1.0</offset_x>
-        <offset_y>0</offset_y>
-        <offset_z>0</offset_z>
-        <axis>1 0 0</axis>
-        <grip_threshold>0.1</grip_threshold>
-        <force_limit>1.0e2</force_limit>
-        <torque_limit>1.0e3</torque_limit>
-        <bend_angle>0.7854</bend_angle>
-        <stiffness>1.0e4</stiffness>
-        <damping>1.0e3</damping>
-        <retry_close>False</retry_close>
-      </surface_gripper>
-    </isaac>
+    </unity>
   </xacro:macro>
 </robot>
